Commit message: maj

File: description/racecar_fixed_wheel.xacro (robot description, xacro)
@@ -67,13 +67,8 @@
     </visual>
   </link>
-  <joint name="base_to_front_left_hinge" type="fixed">
+  <joint name="base_to_front_left_wheel" type="fixed">
     <parent link="base_link"/>
-    <child link="front_left_hinge"/>
+    <child link="front_left_wheel"/>
     <origin xyz="${wheelbase} ${(wheel_length+width)/2} ${wheel_radius}"/>
-  </joint>
-  <link name="front_left_hinge"/>
-  <joint name="front_left_hinge_to_wheel" type="continuous">
-    <parent link="front_left_hinge"/>
-    <child link="front_left_wheel"/>
   </joint>
   <link name="front_left_wheel">
@@ -86,13 +81,8 @@
     </visual>
   </link>
-  <joint name="base_to_front_right_hinge" type="fixed">
+  <joint name="base_to_front_right_wheel" type="fixed">
     <parent link="base_link"/>
-    <child link="front_right_hinge"/>
+    <child link="front_right_wheel"/>
     <origin xyz="${wheelbase} ${-(wheel_length+width)/2} ${wheel_radius}"/>
-  </joint>
-  <link name="front_right_hinge"/>
-  <joint name="front_right_hinge_to_wheel" type="continuous">
-    <parent link="front_right_hinge"/>
-    <child link="front_right_wheel"/>
   </joint>
   <link name="front_right_wheel">

Commit message: maj

File: description/racecar_fixed_wheel.xacro (robot description, xacro)
@@ -11,4 +11,6 @@
   <xacro:property name="laser_height" value="0.05" />
   <xacro:property name="laser_radius" value="0.026" />
+  <xacro:property name="imu_distance_from_base_link" value="0.17" />
+  <xacro:property name="imu_height" value="0.025" />
   <material name="black">
     <color rgba="0.2 0.2 0.2 1."/>
@@ -25,4 +27,11 @@
       <material name="blue"/>
     </visual>
+  </link>
+  <joint name="base_to_imu_model" type="fixed">
+    <parent link="base_link"/>
+    <child link="imu"/>
+    <origin xyz="${imu_distance_from_base_link} 0 ${ground_offset+height+imu_height}"/>
+  </joint>
+  <link name="laser">
   </link>
   <joint name="base_to_laser_model" type="fixed">

Commit message: maj

File: description/racecar_fixed_wheel.xacro (robot description, xacro)
@@ -33,5 +33,5 @@
     <origin xyz="${imu_distance_from_base_link} 0 ${ground_offset+height+imu_height}"/>
   </joint>
-  <link name="laser">
+  <link name="imu">
   </link>
   <joint name="base_to_laser_model" type="fixed">

Commit message: maj

File: description/racecar_fixed_wheel.xacro (robot description, xacro)
@@ -38,5 +38,5 @@
     <parent link="base_link"/>
     <child link="laser"/>
-    <origin xyz="${laser_distance_from_base_link} 0 ${ground_offset+height+(laser_height/2)}"/>
+    <origin rpy="0 0 ${pi/2}" xyz="${laser_distance_from_base_link} 0 ${ground_offset+height+(laser_height/2)}"/>
   </joint>
   <link name="laser">

Commit message: maj

File: description/racecar_fixed_wheel.xacro (robot description, xacro)
@@ -31,5 +31,5 @@
     <parent link="base_link"/>
     <child link="imu"/>
-    <origin xyz="${imu_distance_from_base_link} 0 ${ground_offset+height+imu_height}"/>
+    <origin rpy="0 0 ${-pi/2}" xyz="${imu_distance_from_base_link} 0 ${ground_offset+height+imu_height}"/>
   </joint>
   <link name="imu">
@@ -38,5 +38,5 @@
     <parent link="base_link"/>
     <child link="laser"/>
-    <origin rpy="0 0 ${pi/2}" xyz="${laser_distance_from_base_link} 0 ${ground_offset+height+(laser_height/2)}"/>
+    <origin xyz="${laser_distance_from_base_link} 0 ${ground_offset+height+(laser_height/2)}"/>
   </joint>
   <link name="laser">
